Commit message: changed the environment(world) put it inside a warehouse will change its physical structure too.

File: src/chilax_simulation/urdf/body.urdf.xacro (robot description, xacro)
@@ -1,10 +1,10 @@
 <?xml version="3.0"?>
 <robot xmlns:xacro="http://www.ros.org/wiki/xacro">
-    <xacro:property name="front_body_length" value="0.05" />
-    <xacro:property name="middle_body_length" value="0.21" />
-    <xacro:property name="end_body_length" value="0.05" />
+    <xacro:property name="front_body_length" value="0.03" />
+    <xacro:property name="middle_body_length" value="0.1" />
+    <xacro:property name="end_body_length" value="0.03" />
     <xacro:property name="socket_width" value="0.05" />
     <xacro:property name="socket_length" value="0.07" />
-    <xacro:property name="body_width" value="0.2" />
+    <xacro:property name="body_width" value="0.15" />
     <xacro:property name="body_height" value="0.06" />
     <link name="base_link" />

File: src/chilax_simulation/urdf/leg.urdf.xacro (robot description, xacro)
@@ -1,8 +1,8 @@
 <?xml version="3.0"?>
 <robot xmlns:xacro="http://www.ros.org/wiki/xacro">
-    <xacro:property name="thigh_length" value="0.12" />
-    <xacro:property name="lower_leg_length" value="0.11" />
-    <xacro:property name="leg_width" value="0.04" />
-    <xacro:property name="leg_height" value="0.04" />
+    <xacro:property name="thigh_length" value="0.08" />
+    <xacro:property name="lower_leg_length" value="0.075" />
+    <xacro:property name="leg_width" value="0.03" />
+    <xacro:property name="leg_height" value="0.03" />
     <!-- x_axis = 1 means front, -1 means back and y_axis = 1 means left, -1 means right -->
     <xacro:macro name="create_leg" params="prefix">
